File: pcb/pmod_spdif/pmod_spdif.sch (KiCad schematic (older format))
At the start: 17 parts, among them J1 PMOD, J2 Conn_01x06_Male, U1 74HC04, U2 CAT3200-5, U3 TOTX1350(F), U4 SN74LVC1T45DBV

Commit message: pmod_spdif v2. Only cosmetic changes.
Parts:
- R4: value R -> 1K
Other:
- note added: "0 Ohm resistor for easy\npatching if something \ndoesn't work."
- note added: "PMOD 3V3 to 5V.\nThe HC04 buffers have Vih of 3.6V when \npowered at 5V, so regular 3V3 IOs won't do."
- note added: "Parallel HC04 drivers, copied from \nTOTX1350(F) datasheet.\nThere might be buffers with 3V3 input\nand 5V output that can drive the TOSLINK\nLED, but I didn't want to take any chances\nand just used the reference design."
- note added: "TOTX1350(F) requires 5V."
Changed lines of the file:
@@
 P 3000 2850
 F 0 "R4" V 3100 2800 50  0000 C CNN
-F 1 "R" V 2900 2800 50  0000 C CNN
+F 1 "1K" V 2900 2800 50  0000 C CNN
 F 2 "Resistor_SMD:R_0603_1608Metric_Pad1.05x0.95mm_HandSolder" V 2930 2850 50  0001 C CNN
 F 3 "~" H 3000 2850 50  0001 C CNN
@@
 NoConn ~ 1250 1450
 NoConn ~ 1250 1550
+Text Notes 5350 2000 0    50   ~ 0
+Parallel HC04 drivers, copied from \nTOTX1350(F) datasheet.\nThere might be buffers with 3V3 input\nand 5V output that can drive the TOSLINK\nLED, but I didn't want to take any chances\nand just used the reference design.
+Text Notes 4250 2400 0    50   ~ 0
+0 Ohm resistor for easy\npatching if something \ndoesn't work.
+Text Notes 6150 3600 0    50   ~ 0
+TOTX1350(F)  requires 5V.
+Text Notes 2400 3550 0    50   ~ 0
+PMOD 3V3 to 5V.\nThe HC04 buffers have Vih of 3.6V when \npowered at 5V, so regular 3V3 IOs won't do.
 $EndSCHEMATC

Commit message: Update documentation.
Other:
- note added: "Route some unused PMOD signals to \na generic connector.\n"
- note added: "TOTX1350(F) requires 5V. Create\nthat from 3V3."
- note removed: "TOTX1350(F) requires 5V."
- moved on the sheet: C1, C2, C3, C4, C6, J1, J2, R1, R2, R3, R4, R5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
